File: KiCad/EnergyMonitor.kicad_pcb (KiCad board)
At the start: 2 copper layers, 40 parts, among them J1 Conn_01x02, J10 4P4C, J5 Conn_01x02, J6 Conn_01x02, J7 Conn_01x02, J9 Conn_01x04, U3 HT7333

Commit message: pcb footprints
Parts:
- added D5: ESD5Z3.3T1G, Diode_SMD:D_SOD-523, F.Cu at (224.8, 128.3)
- added J2: AudioJack3_Ground_SwitchTR, MyFootprints:3.5mm_5_Pin_Socket_PCB_Mount, F.Cu at (162.6, 58.4)
- added J3: AudioJack3_Ground_SwitchTR, MyFootprints:3.5mm_5_Pin_Socket_PCB_Mount, F.Cu at (175.3, 58.4)
- added J4: AudioJack3_Ground_SwitchTR, MyFootprints:3.5mm_5_Pin_Socket_PCB_Mount, F.Cu at (188.0, 58.4)
- added J8: Barrel_Jack_Switch, MyFootprints:DC_Barrel_Jack_Socket, F.Cu at (149.9, 58.4)
- added U2: ESP32_D1_MINI, MyFootprints:ESP32_D1_MINI, F.Cu at (101.6, 104.1)
- moved J10 94.1 mm to (121.9, 66.0)
- moved R4 59.9 mm to (167.6, 96.3)
- moved R7 59.9 mm to (183.4, 86.1)
- moved C1 59.9 mm to (149.9, 97.8)
- moved C10 59.9 mm to (177.6, 79.6)
- moved C2 59.9 mm to (168.3, 86.8)
- moved C3 59.9 mm to (172.1, 93.4)
- moved C4 59.9 mm to (167.7, 93.4)
- moved C5 59.9 mm to (173.3, 90.0)
- moved C6 59.9 mm to (168.3, 90.2)
- moved C7 59.9 mm to (173.9, 86.8)
- moved C8 59.9 mm to (179.6, 83.0)
- moved C9 59.9 mm to (179.0, 86.2)
- moved D2 59.9 mm to (184.9, 91.8)
- moved D3 59.9 mm to (147.2, 102.4)
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
Commit message: pcb layout
Parts:
- moved J2 72.8 mm to (154.9, 130.8), turned to 270 degrees
- moved J8 65.4 mm to (123.2, 118.1), turned to 180 degrees
- moved R11 64.8 mm to (146.7, 131.4)
- moved R12 63.5 mm to (146.7, 133.3), turned to 180 degrees
- moved J4 60.6 mm to (137.2, 91.4), turned to 270 degrees
- moved J3 59.5 mm to (137.2, 104.1), turned to 270 degrees
- moved D2 58.7 mm to (242.6, 102.9)
- moved R2 58.6 mm to (146.7, 125.7)
- moved J5 54.6 mm to (142.9, 128.9), turned to 180 degrees
- moved C10 51.1 mm to (227.1, 92.3)
- moved C2 51.1 mm to (217.8, 99.5)
- moved C5 51.1 mm to (222.8, 102.7)
- moved C7 51.1 mm to (223.4, 99.5)
- moved C8 51.1 mm to (229.1, 95.7)
- moved C9 51.1 mm to (228.5, 98.9)
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Routing:
- net Net-(C3-Pad2): track 0.00 -> 27.9 mm
- net Net-(C3-Pad1): track 0.00 -> 13.4 mm
- net Net-(J5-Pad2): track 0.00 -> 5.07 mm

Commit message: circuit design & pcb layout
Parts:
- removed the J7 at (212.6, 105.2)
- added D1: IN4148, Diode_THT:D_DO-35_SOD27_P7.62mm_Horizontal, F.Cu at (158.1, 120.7)
- added J1: Conn_01x04, Connector_PinHeader_2.54mm:PinHeader_1x04_P2.54mm_Vertical, F.Cu at (95.2, 99.7)
- added J10: AudioJack3_Ground_Switch_5_pin, MyFootprints:3.5mm_5_Pin_Socket_PCB_Mount, F.Cu at (124.5, 120.0)
- added J14: Conn_01x04, Connector_JST:JST_SH_SM04B-SRSS-TB_1x04-1MP_P1.00mm_Horizontal, F.Cu at (76.2, 137.8)
- added J8: AudioJack3_Ground_Switch_5_pin, MyFootprints:3.5mm_5_Pin_Socket_PCB_Mount, F.Cu at (111.8, 120.0)
- added J9: AudioJack3_Ground_Switch_5_pin, MyFootprints:3.5mm_5_Pin_Socket_PCB_Mount, F.Cu at (99.1, 120.0)
- added R1: 56R 0.25W, Resistor_SMD:R_1206_3216Metric, F.Cu at (165.4, 113.7)
- added R10: 22R, Resistor_SMD:R_1206_3216Metric, F.Cu at (127.3, 107.3)
- added R11: 39R, Resistor_SMD:R_1206_3216Metric, F.Cu at (127.3, 104.8)
- added R12: 62R, Resistor_SMD:R_1206_3216Metric, F.Cu at (127.3, 102.2)
- added R13: 120R, Resistor_SMD:R_1206_3216Metric, F.Cu at (127.3, 99.7)
- added R8: 62R, Resistor_SMD:R_1206_3216Metric, F.Cu at (114.6, 102.2)
- added R9: 120R, Resistor_SMD:R_1206_3216Metric, F.Cu at (114.6, 99.7)
- J16: renamed from J10; footprint MyFootprints:RJ6_4P4C_small_I2C -> MyFootprints:RJ6_4P4C_small_I2C_UM10204
- J2, J3, J4: value AudioJack3_Ground_SwitchTR -> Conn_01x04; footprint MyFootprints:3.5mm_5_Pin_Socket_PCB_Mount -> Connector_PinHeader_2.54mm:PinHeader_1x04_P2.54mm_Vertical
- J5, J6: value Conn_01x02 -> Conn_01x04; footprint Connector_PinHeader_2.54mm:PinHeader_1x02_P2.54mm_Vertical -> Connector_PinHeader_2.54mm:PinHeader_1x04_P2.54mm_Vertical
- R2, R6: footprint Resistor_SMD:R_0805_2012Metric -> Resistor_SMD:R_1206_3216Metric
- R3, R7: value 22R -> 39R; footprint Resistor_SMD:R_0805_2012Metric -> Resistor_SMD:R_1206_3216Metric
- R4: value 22R -> 62R; footprint Resistor_SMD:R_0805_2012Metric -> Resistor_SMD:R_1206_3216Metric
- R5: value 22R -> 120R; footprint Resistor_SMD:R_0805_2012Metric -> Resistor_SMD:R_1206_3216Metric
- moved D2 147.9 mm to (94.9, 94.3)
- moved R3 131.0 mm to (101.9, 104.8), turned to 180 degrees
- moved R21 126.9 mm to (111.1, 111.4), turned to 270 degrees
- moved R7 118.5 mm to (114.6, 104.8), turned to 180 degrees
- moved R17 118.2 mm to (108.0, 110.5)
- moved R4 115.5 mm to (101.9, 102.2), turned to 180 degrees
- moved R23 114.3 mm to (123.8, 111.4), turned to 270 degrees
- moved R6 114.0 mm to (114.6, 107.3), turned to 180 degrees
- moved R22 113.1 mm to (113.0, 111.4), turned to 270 degrees
- moved C4 109.4 mm to (108.0, 112.4)
- moved C7 108.2 mm to (115.9, 111.1), turned to 270 degrees
- moved R24 105.0 mm to (125.7, 111.4), turned to 270 degrees
- moved C5 102.6 mm to (120.7, 112.4)
- moved C8 101.7 mm to (128.6, 111.1), turned to 270 degrees
- moved R18 96.3 mm to (120.7, 110.5)
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- renumbered J8 to J13, J9 to J15, J1 to J7, R8 to R16, R9 to R17, R10 to R18, R11 to R19, R12 to R20, R13 to R21, R14 to R22, R15 to R23, R16 to R24, R17 to R25, R18 to R26, R19 to R27, R20 to R28, R21 to R29, U2 to U1, U3 to U2
Connections:
- C3 pad 1: Net-(C3-Pad1) -> RB1
- C3 pad 2: Net-(C3-Pad2) -> TB1
- C4 pad 1: Net-(C4-Pad1) -> RB2
- C4 pad 2: Net-(C4-Pad2) -> TB2
- C5 pad 1: Net-(C5-Pad1) -> RB3
- C5 pad 2: Net-(C5-Pad2) -> TB3
- C6 pad 1: Net-(C3-Pad2) -> TB1
- C7 pad 1: Net-(C4-Pad2) -> TB2
- C8 pad 1: Net-(C5-Pad2) -> TB3
- J5 pad 1: Net-(C3-Pad1) -> Net-(J5-Pad1)
- J6 pad 1: Net-(C4-Pad1) -> Net-(J6-Pad1)
- R16 pad 2: Net-(C3-Pad1) -> RB1
- R17 pad 2: Net-(C4-Pad1) -> RB2
- R18 pad 2: Net-(C5-Pad1) -> RB3
- R19 pad 2: Net-(C3-Pad2) -> TB1
- R2 pad 1: Net-(J5-Pad2) -> TB1
- R2 pad 2: Net-(C3-Pad2) -> Net-(J4-Pad4)
- R20 pad 1: Net-(C3-Pad2) -> TB1
- R21 pad 2: Net-(C4-Pad2) -> TB2
- R22 pad 1: Net-(C4-Pad2) -> TB2
- R23 pad 2: Net-(C5-Pad2) -> TB3
- R24 pad 1: Net-(C5-Pad2) -> TB3
- R3 pad 1: Net-(J6-Pad2) -> TB1
- R3 pad 2: Net-(C4-Pad2) -> Net-(J4-Pad3)
- R4 pad 1: Net-(J7-Pad2) -> TB1
- R4 pad 2: Net-(C5-Pad2) -> Net-(J4-Pad2)
- R5 pad 1: Net-(J5-Pad2) -> TB1
- R5 pad 2: Net-(C3-Pad2) -> Net-(J4-Pad1)
- R6 pad 1: Net-(J6-Pad2) -> TB2
- R6 pad 2: Net-(C4-Pad2) -> Net-(J5-Pad4)
- R7 pad 1: Net-(J7-Pad2) -> TB2
- R7 pad 2: Net-(C5-Pad2) -> Net-(J5-Pad3)
- U1 pad 10: SPI_MISO -> (no net)
- U1 pad 12: SPI_MOSI -> (no net)
- U1 pad 13: Net-(U2-Pad13) -> (no net)
- U1 pad 14: SPI_CS -> (no net)
- U1 pad 15: Net-(U2-Pad15) -> (no net)
- U1 pad 17: Net-(U2-Pad17) -> (no net)
- U1 pad 18: Net-(U2-Pad18) -> (no net)
- U1 pad 19: Net-(U2-Pad19) -> (no net)
- U1 pad 2: Net-(U2-Pad2) -> (no net)
- U1 pad 20: Net-(U2-Pad20) -> (no net)
- U1 pad 21: Net-(U2-Pad21) -> (no net)
- U1 pad 22: Net-(U2-Pad22) -> (no net)
- U1 pad 23: Net-(U2-Pad23) -> (no net)
- U1 pad 24: Net-(U2-Pad24) -> (no net)
- U1 pad 25: Net-(U2-Pad25) -> (no net)
- U1 pad 26: Net-(U2-Pad26) -> (no net)
- U1 pad 27: Net-(U2-Pad27) -> (no net)
- U1 pad 29: Net-(U2-Pad29) -> (no net)
- U1 pad 3: Net-(U2-Pad3) -> (no net)
- U1 pad 30: Net-(U2-Pad30) -> (no net)
- U1 pad 31: Net-(U2-Pad31) -> (no net)
- U1 pad 32: Net-(U2-Pad32) -> (no net)
- U1 pad 35: Net-(U2-Pad35) -> (no net)
- U1 pad 37: Net-(U2-Pad37) -> (no net)
- U1 pad 38: Net-(U2-Pad38) -> (no net)
- U1 pad 4: Net-(U2-Pad4) -> (no net)
- U1 pad 40: Net-(U2-Pad40) -> (no net)
- U1 pad 5: Net-(U2-Pad5) -> (no net)
- U1 pad 6: Net-(U2-Pad6) -> (no net)
- U1 pad 8: SPI_CLK -> (no net)
Routing:
- net Net-(C3-Pad2): track 27.9 -> 0.00 mm
- net TB1: track 0.00 -> 25.4 mm
- net TB2: track 0.00 -> 25.4 mm
- net TB3: track 0.00 -> 25.3 mm
- net ADC1_CH5: track 0.00 -> 23.8 mm
- net RB1: track 0.00 -> 17.8 mm
- net RB3: track 0.00 -> 17.7 mm
- net RB2: track 0.00 -> 17.7 mm
- net Net-(C3-Pad1): track 13.4 -> 0.00 mm
- net Net-(J6-Pad4): track 0.00 -> 2.67 mm
- net Net-(J6-Pad3): track 0.00 -> 2.67 mm
- net Net-(J6-Pad2): track 0.00 -> 2.67 mm
- net Net-(J6-Pad1): track 0.00 -> 2.67 mm
- net Net-(J5-Pad4): track 0.00 -> 2.67 mm
- net Net-(J5-Pad3): track 0.00 -> 2.67 mm
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Other:
- board outline added: 99.7 x 49.5 mm
- board text added: "120R 62R 39R 22R"
- board text added: "16A 32A 50A 95A"
- board text added: "9VAC"
- board text added: "Current Transformers YHDC SCT-013-00 CT"
- board text added: "remove jumper if CT sensor has built-in burden resistor"

Commit message: circuit design & pcb layout
Parts:
- moved D5 103.3 mm to (82.5, 92.1)
- moved J16 76.8 mm to (74.9, 121.3), turned to 180 degrees
- moved R26 75.5 mm to (124.8, 84.1)
- moved R29 70.4 mm to (131.4, 87.0), turned to 270 degrees
- moved R27 68.2 mm to (127.6, 87.0), turned to 270 degrees
- moved R28 65.9 mm to (129.5, 87.0), turned to 270 degrees
- moved R25 64.8 mm to (125.7, 87.0), turned to 90 degrees
- moved C9 60.8 mm to (123.8, 87.0), turned to 270 degrees
- moved J15 58.5 mm to (86.4, 122.2), turned to 180 degrees
- moved C10 54.3 mm to (134.3, 86.7), turned to 270 degrees
- moved J7 44.8 mm to (136.8, 99.7), turned to 180 degrees
- moved D4 38.1 mm to (82.5, 94.0)
- moved C1 26.4 mm to (139.1, 104.8), turned to 180 degrees
- moved D3 24.5 mm to (82.5, 95.9)
- moved J14 23.6 mm to (60.3, 120.3)
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- renumbered U1 to ESP32
Routing:
- net I2C_SCL: track 0.00 -> 64.5 mm
- net I2C_SDA: track 0.00 -> 39.8 mm
- net +3V3: track 0.00 -> 29.4 mm
- net ADC1_CH5: track 23.8 -> 0.00 mm
Other:
- board text added: "3V3"
- board text added: "AC-AC measurement"
- board text added: "ESP32"
- board text added: "GND"
- board text added: "I2C"
- board text added: "SCL"
- board text added: "SDA"
- board text added: "UM10204"
- board text added: "Wemos"
- board text added: "remove jumber if powered by USB"

Commit message: circuit design & pcb layout
Other:
- board text added: "3V3 DC"
- board text added: "AC sampling"
- board text added: "ESD"
- board text added: "remove jumper if powered by USB"
- board text removed: "AC-AC measurement"
- board text removed: "remove jumber if powered by USB"
Changed lines of the file:
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@@
   (general
     (thickness 1.6)
-    (drawings 34)
+    (drawings 36)
     (tracks 132)
     (zones 0)
@@
     (pad 4 thru_hole circle (at -11.43 -8.89 270) (size 1.524 1.524) (drill 0.762) (layers *.Cu *.Mask))
     (pad 2 thru_hole circle (at -11.43 -11.43 270) (size 1.524 1.524) (drill 0.762) (layers *.Cu *.Mask))
+    (model ${KISYS3DMOD}/Connector_PinSocket_2.54mm.3dshapes/PinSocket_1x10_P2.54mm_Vertical.wrl
+      (offset (xyz -14 11.5 0))
+      (scale (xyz 1 1 1))
+      (rotate (xyz 0 0 0))
+    )
+    (model ${KISYS3DMOD}/Connector_PinSocket_2.54mm.3dshapes/PinSocket_1x10_P2.54mm_Vertical.wrl
+      (offset (xyz -11.5 11.5 0))
+      (scale (xyz 1 1 1))
+      (rotate (xyz 0 0 0))
+    )
+    (model ${KISYS3DMOD}/Connector_PinSocket_2.54mm.3dshapes/PinSocket_1x10_P2.54mm_Vertical.wrl
+      (offset (xyz 14 11.5 0))
+      (scale (xyz 1 1 1))
+      (rotate (xyz 0 0 0))
+    )
+    (model ${KISYS3DMOD}/Connector_PinSocket_2.54mm.3dshapes/PinSocket_1x10_P2.54mm_Vertical.wrl
+      (offset (xyz 11.5 11.5 0))
+      (scale (xyz 1 1 1))
+      (rotate (xyz 0 0 0))
+    )
   )
   (module MyFootprints:DC_Barrel_Jack_Socket (layer F.Cu)
@@
       (effects (font (size 1 1) (thickness 0.15)))
     )
-    (fp_text value Conn_01x02 (at 0 4.87) (layer F.Fab)
+    (fp_text value Conn_01x02 (at 0 4.87) (layer F.Fab) hide
       (effects (font (size 1 1) (thickness 0.15)))
     )
@@
     )
   )
-  (gr_text "remove jumber if\npowered by USB" (at 140.6525 93.0275) (layer F.SilkS)
+  (gr_text "3V3\nDC" (at 133.6675 97.155) (layer F.SilkS)
     (effects (font (size 1 1) (thickness 0.15)))
   )
-  (gr_text "AC-AC\nmeasurement" (at 132.715 81.5975) (layer F.SilkS)
+  (gr_text ESD (at 82.55 90.17) (layer F.SilkS)
     (effects (font (size 1 1) (thickness 0.15)))
   )
+  (gr_text "remove jumper if\npowered by USB" (at 140.6525 92.71) (layer F.SilkS)
+    (effects (font (size 1 1) (thickness 0.15)))
+  )
+  (gr_text "AC\nsampling" (at 131.7625 81.5975) (layer F.SilkS)
+    (effects (font (size 1 1) (thickness 0.15)))
+  )

Commit message: create 3D models for PCB components
Parts:
- moved J13 0.32 mm to (141.0, 120.3)
- renumbered ESP32 to U1
Connections:
- J10 pad RN: (no net) -> Net-(J10-PadRN)
- J8 pad RN: (no net) -> Net-(J8-PadRN)
- J9 pad RN: (no net) -> Net-(J9-PadRN)
- U1 pad 10: (no net) -> SPI_MISO
- U1 pad 12: (no net) -> SPI_MOSI
- U1 pad 13: (no net) -> Net-(U1-Pad13)
- U1 pad 14: (no net) -> SPI_CS
- U1 pad 15: (no net) -> Net-(U1-Pad15)
- U1 pad 17: (no net) -> Net-(U1-Pad17)
- U1 pad 18: (no net) -> Net-(U1-Pad18)
- U1 pad 19: (no net) -> Net-(U1-Pad19)
- U1 pad 2: (no net) -> Net-(U1-Pad2)
- U1 pad 20: (no net) -> Net-(U1-Pad20)
- U1 pad 21: (no net) -> Net-(U1-Pad21)
- U1 pad 22: (no net) -> Net-(U1-Pad22)
- U1 pad 23: (no net) -> Net-(U1-Pad23)
- U1 pad 24: (no net) -> Net-(U1-Pad24)
- U1 pad 25: (no net) -> Net-(U1-Pad25)
- U1 pad 26: (no net) -> Net-(U1-Pad26)
- U1 pad 27: (no net) -> Net-(U1-Pad27)
- U1 pad 29: (no net) -> Net-(U1-Pad29)
- U1 pad 3: (no net) -> Net-(U1-Pad3)
- U1 pad 30: (no net) -> Net-(U1-Pad30)
- U1 pad 31: (no net) -> Net-(U1-Pad31)
- U1 pad 32: (no net) -> Net-(U1-Pad32)
- U1 pad 35: (no net) -> Net-(U1-Pad35)
- U1 pad 37: (no net) -> Net-(U1-Pad37)
- U1 pad 38: (no net) -> Net-(U1-Pad38)
- U1 pad 4: (no net) -> Net-(U1-Pad4)
- U1 pad 40: (no net) -> Net-(U1-Pad40)
- U1 pad 5: (no net) -> Net-(U1-Pad5)
- U1 pad 6: (no net) -> Net-(U1-Pad6)
- U1 pad 8: (no net) -> SPI_CLK
Routing:
- net RB1: track 17.8 -> 18.5 mm

Commit message: circuit design & pcb layout
Parts:
- added D6: LED, LED_SMD:LED_0805_2012Metric, F.Cu at (104.1, 81.0)
- added H1: MountingHole, MountingHole:MountingHole_2.2mm_M2_Pad_Via, F.Cu at (146.7, 78.7)
- added H2: MountingHole, MountingHole:MountingHole_2.2mm_M2_Pad_Via, F.Cu at (53.3, 78.7)
- added H3: MountingHole, MountingHole:MountingHole_2.2mm_M2_Pad_Via, F.Cu at (53.3, 121.9)
- added H4: MountingHole, MountingHole:MountingHole_2.2mm_M2_Pad_Via, F.Cu at (146.7, 121.9)
- added J11: Conn_01x02, Connector_PinHeader_2.54mm:PinHeader_1x02_P2.54mm_Vertical, F.Cu at (141.0, 92.1)
- added R14: 4K7, LED_SMD:LED_0805_2012Metric, F.Cu at (108.0, 81.0)
- added TP1: TestPoint_Probe, TestPoint:TestPoint_Loop_D2.50mm_Drill1.0mm_LowProfile, F.Cu at (91.4, 100.0)
- added TP2: TestPoint_Probe, TestPoint:TestPoint_Loop_D2.50mm_Drill1.0mm_LowProfile, F.Cu at (91.4, 94.9)
- added TP3: TestPoint_Probe, TestPoint:TestPoint_Loop_D2.50mm_Drill1.0mm_LowProfile, F.Cu at (91.4, 89.9)
- added TP4: TestPoint_Probe, TestPoint:TestPoint_Loop_D2.50mm_Drill1.0mm_LowProfile, F.Cu at (91.4, 84.8)
- added TP5: TestPoint_Probe, TestPoint:TestPoint_Loop_D2.50mm_Drill1.0mm_LowProfile, F.Cu at (91.4, 105.1)
- moved D1 25.6 mm to (137.5, 85.1), turned to 270 degrees
- moved C9 23.8 mm to (136.2, 107.3), turned to 180 degrees
- moved R1 23.3 mm to (132.7, 85.1), turned to 0 degrees
- moved C10 22.3 mm to (144.1, 106.7)
- moved R28 22.0 mm to (139.4, 106.7)
- moved R29 22.0 mm to (141.3, 106.7)
- moved C2 21.6 mm to (126.7, 87.6), turned to 0 degrees
- moved R25 21.2 mm to (136.2, 105.4), turned to 180 degrees
- moved R26 20.9 mm to (136.2, 101.6)
- moved R27 18.6 mm to (136.2, 103.5), turned to 0 degrees
- moved J7 17.6 mm to (128.0, 84.5), turned to 270 degrees
- moved U2 16.1 mm to (126.7, 91.8), turned to 270 degrees
- moved C1 15.1 mm to (132.7, 91.1), turned to 270 degrees
- moved J13 1.91 mm to (139.1, 120.3)
- moved U1 1.59 mm to (68.9, 94.9)
Connections:
- D1 pad 2: 9V_AC -> Net-(D1-Pad2)
- J10 pad RN: Net-(J10-PadRN) -> (no net)
- J8 pad RN: Net-(J8-PadRN) -> (no net)
- J9 pad RN: Net-(J9-PadRN) -> (no net)
- U1 pad 10: SPI_MISO -> (no net)
- U1 pad 12: SPI_MOSI -> (no net)
- U1 pad 13: Net-(U1-Pad13) -> (no net)
- U1 pad 14: SPI_CS -> (no net)
- U1 pad 15: Net-(U1-Pad15) -> (no net)
- U1 pad 17: Net-(U1-Pad17) -> (no net)
- U1 pad 18: Net-(U1-Pad18) -> (no net)
- U1 pad 19: Net-(U1-Pad19) -> (no net)
- U1 pad 2: Net-(U1-Pad2) -> (no net)
- U1 pad 20: Net-(U1-Pad20) -> (no net)
- U1 pad 21: Net-(U1-Pad21) -> (no net)
- U1 pad 22: Net-(U1-Pad22) -> (no net)
- U1 pad 23: Net-(U1-Pad23) -> (no net)
- U1 pad 24: Net-(U1-Pad24) -> (no net)
- U1 pad 25: Net-(U1-Pad25) -> (no net)
- U1 pad 26: Net-(U1-Pad26) -> (no net)
- U1 pad 27: Net-(U1-Pad27) -> (no net)
- U1 pad 29: Net-(U1-Pad29) -> (no net)
- U1 pad 3: Net-(U1-Pad3) -> (no net)
- U1 pad 30: Net-(U1-Pad30) -> (no net)
- U1 pad 31: Net-(U1-Pad31) -> (no net)
- U1 pad 32: Net-(U1-Pad32) -> (no net)
- U1 pad 35: Net-(U1-Pad35) -> (no net)
- U1 pad 37: Net-(U1-Pad37) -> (no net)
- U1 pad 38: Net-(U1-Pad38) -> (no net)
- U1 pad 4: Net-(U1-Pad4) -> (no net)
- U1 pad 40: Net-(U1-Pad40) -> (no net)
- U1 pad 5: Net-(U1-Pad5) -> (no net)
- U1 pad 6: Net-(U1-Pad6) -> (no net)
- U1 pad 8: SPI_CLK -> (no net)
Routing:
- net Net-(D6-Pad2): track 0.00 -> 1.94 mm
- net I2C_SCL: track 64.5 -> 62.9 mm
Other:
- outline, holes or cut-outs redrawn
- board text added: "9V AC"
- board text added: "AC voltage ADC"
- board text added: "I1"
- board text added: "I2"
- board text added: "I3"
- board text added: "V"
- board text added: "remove jumper on USB power"
- board text removed: "AC sampling"
- board text removed: "remove jumper if powered by USB"

Commit message: circuit design & pcb layout
Parts:
- R14: footprint LED_SMD:LED_0805_2012Metric -> Resistor_SMD:R_0805_2012Metric
Other:
- board text added: "sample rate 2500 Hz"
Changed lines of the file:
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@@
   (general
     (thickness 1.6)
-    (drawings 54)
+    (drawings 55)
     (tracks 135)
     (zones 0)
@@
     (add_net TB3)
   )
+  (module Resistor_SMD:R_0805_2012Metric (layer F.Cu)
+    (at 107.95 80.9625 180)
+    (descr "Resistor SMD 0805 (2012 Metric), square (rectangular) end terminal, IPC_7351 nominal, (Body size source: IPC-SM-782 page 72, https://www.pcb-3d.com/wordpress/wp-content/uploads/ipc-sm-782a_amendment_1_and_2.pdf), generated with kicad-footprint-generator")
+    (tags resistor)
+    (attr smd)
+    (fp_text reference R14 (at 0 -1.65) (layer F.SilkS) hide
+      (effects (font (size 1 1) (thickness 0.15)))
+    )
+    (fp_text value 4K7 (at 0 1.65) (layer F.Fab)
+      (effects (font (size 1 1) (thickness 0.15)))
+    )
+    (fp_text user %R (at 0 0) (layer F.Fab)
+      (effects (font (size 0.5 0.5) (thickness 0.08)))
+    )
+    (fp_line (start -1 0.625) (end -1 -0.625) (layer F.Fab) (width 0.1))
+    (fp_line (start -1 -0.625) (end 1 -0.625) (layer F.Fab) (width 0.1))
+    (fp_line (start 1 -0.625) (end 1 0.625) (layer F.Fab) (width 0.1))
+    (fp_line (start 1 0.625) (end -1 0.625) (layer F.Fab) (width 0.1))
+    (fp_line (start -0.227064 -0.735) (end 0.227064 -0.735) (layer F.SilkS) (width 0.12))
+    (fp_line (start -0.227064 0.735) (end 0.227064 0.735) (layer F.SilkS) (width 0.12))
+    (fp_line (start -1.68 0.95) (end -1.68 -0.95) (layer F.CrtYd) (width 0.05))
+    (fp_line (start -1.68 -0.95) (end 1.68 -0.95) (layer F.CrtYd) (width 0.05))
+    (fp_line (start 1.68 -0.95) (end 1.68 0.95) (layer F.CrtYd) (width 0.05))
+    (fp_line (start 1.68 0.95) (end -1.68 0.95) (layer F.CrtYd) (width 0.05))
+    (pad 2 smd roundrect (at 0.9125 0 180) (size 1.025 1.4) (layers F.Cu F.Paste F.Mask) (roundrect_rratio 0.243902)
+      (net 36 "Net-(D6-Pad2)"))
+    (pad 1 smd roundrect (at -0.9125 0 180) (size 1.025 1.4) (layers F.Cu F.Paste F.Mask) (roundrect_rratio 0.243902)
+      (net 11 +3V3))
+    (model ${KISYS3DMOD}/Resistor_SMD.3dshapes/R_0805_2012Metric.wrl
+      (at (xyz 0 0 0))
+      (scale (xyz 1 1 1))
+      (rotate (xyz 0 0 0))
+    )
+  )
   (module LED_SMD:LED_0805_2012Metric (layer F.Cu)
-    (at 107.95 80.9625 180)
+    (at 104.14 80.9625)
     (descr "LED SMD 0805 (2012 Metric), square (rectangular) end terminal, IPC_7351 nominal, (Body size source: https://docs.google.com/spreadsheets/d/1BsfQQcO9C6DZCsRaXUlFlo91Tg2WpOkGARC1WS5S8t0/edit?usp=sharing), generated with kicad-footprint-generator")
     (tags LED)
     (attr smd)
-    (fp_text reference R14 (at 0 -1.65) (layer F.SilkS) hide
-      (effects (font (size 1 1) (thickness 0.15)))
-    )
-    (fp_text value 4K7 (at 0 -0.3175) (layer F.Fab)
-      (effects (font (size 0.3 0.3) (thickness 0.05)))
-    )
-    (fp_text user %R (at 0.005 0.3175) (layer F.Fab)
+    (fp_text reference D6 (at 0 -1.65) (layer F.SilkS) hide
+      (effects (font (size 1 1) (thickness 0.15)))
+    )
+    (fp_text value LED (at 0 0.3175) (layer F.Fab)
       (effects (font (size 0.3 0.3) (thickness 0.05)))
     )
@@
     (fp_line (start 1.68 -0.95) (end 1.68 0.95) (layer F.CrtYd) (width 0.05))
     (fp_line (start 1.68 0.95) (end -1.68 0.95) (layer F.CrtYd) (width 0.05))
-    (pad 2 smd roundrect (at 0.9375 0 180) (size 0.975 1.4) (layers F.Cu F.Paste F.Mask) (roundrect_rratio 0.25)
-      (net 36 "Net-(D6-Pad2)"))
-    (pad 1 smd roundrect (at -0.9375 0 180) (size 0.975 1.4) (layers F.Cu F.Paste F.Mask) (roundrect_rratio 0.25)
-      (net 11 +3V3))
-    (model ${KISYS3DMOD}/LED_SMD.3dshapes/LED_0805_2012Metric.wrl
-      (at (xyz 0 0 0))
-      (scale (xyz 1 1 1))
-      (rotate (xyz 0 0 0))
-    )
-  )
-  (module LED_SMD:LED_0805_2012Metric (layer F.Cu)
-    (at 104.14 80.9625)
-    (descr "LED SMD 0805 (2012 Metric), square (rectangular) end terminal, IPC_7351 nominal, (Body size source: https://docs.google.com/spreadsheets/d/1BsfQQcO9C6DZCsRaXUlFlo91Tg2WpOkGARC1WS5S8t0/edit?usp=sharing), generated with kicad-footprint-generator")
-    (tags LED)
-    (attr smd)
-    (fp_text reference D6 (at 0 -1.65) (layer F.SilkS) hide
-      (effects (font (size 1 1) (thickness 0.15)))
-    )
-    (fp_text value LED (at 0 0.3175) (layer F.Fab)
-      (effects (font (size 0.3 0.3) (thickness 0.05)))
-    )
     (fp_text user %R (at 0 -0.3175) (layer F.Fab)
       (effects (font (size 0.3 0.3) (thickness 0.05)))
     )
-    (fp_line (start 1 -0.6) (end -0.7 -0.6) (layer F.Fab) (width 0.1))
-    (fp_line (start -0.7 -0.6) (end -1 -0.3) (layer F.Fab) (width 0.1))
-    (fp_line (start -1 -0.3) (end -1 0.6) (layer F.Fab) (width 0.1))
-    (fp_line (start -1 0.6) (end 1 0.6) (layer F.Fab) (width 0.1))
-    (fp_line (start 1 0.6) (end 1 -0.6) (layer F.Fab) (width 0.1))
-    (fp_line (start 1 -0.96) (end -1.685 -0.96) (layer F.SilkS) (width 0.12))
-    (fp_line (start -1.685 -0.96) (end -1.685 0.96) (layer F.SilkS) (width 0.12))
-    (fp_line (start -1.685 0.96) (end 1 0.96) (layer F.SilkS) (width 0.12))
-    (fp_line (start -1.68 0.95) (end -1.68 -0.95) (layer F.CrtYd) (width 0.05))
-    (fp_line (start -1.68 -0.95) (end 1.68 -0.95) (layer F.CrtYd) (width 0.05))
-    (fp_line (start 1.68 -0.95) (end 1.68 0.95) (layer F.CrtYd) (width 0.05))
-    (fp_line (start 1.68 0.95) (end -1.68 0.95) (layer F.CrtYd) (width 0.05))
     (pad 2 smd roundrect (at 0.9375 0) (size 0.975 1.4) (layers F.Cu F.Paste F.Mask) (roundrect_rratio 0.25)
       (net 36 "Net-(D6-Pad2)"))
@@
     )
   )
+  (gr_text "sample rate\n2500 Hz" (at 91.7575 80.01) (layer F.SilkS)
+    (effects (font (size 1 1) (thickness 0.15)))
+  )
   (gr_line (start 136.2075 81.915) (end 129.2225 81.915) (layer F.SilkS) (width 0.12))
