File: KiCad/v1.0/EnergyMonitor.sch (KiCad schematic (older format))
At the start: 79 parts, among them J1 Conn_01x04, J10 AudioJack3_Ground_Switch_5_pin, J11 Conn_01x02, J12 Conn_01x04, J13 Barrel_Jack_Switch, J14 Conn_01x04, J15 Conn_01x04, J16 4P4C, J17 Conn_01x06, J2 Conn_01x04, J3 Conn_01x04, J4 Conn_01x04, J5 Conn_01x04, J6 Conn_01x04, J7 Conn_01x02, J8 AudioJack3_Ground_Switch_5_pin, J9 AudioJack3_Ground_Switch_5_pin, U1 ESP32_D1_MINI, U2 HT7333

Commit message: pcb fabrication and assembly, case design
Other:
- note added: "GPIO\n40mA source\n28mA sink\n1.5A total"
Changed lines of the file:
@@
 Sheet 1 1
 Title "ESP32 Energy Monitor"
-Date "2021-09-25"
+Date "2021-10-02"
 Rev "v1.0"
 Comp ""
@@
 NoConn ~ 5100 5000
 NoConn ~ 2450 2525
+Text Notes 2725 1600 0    50   ~ 0
+GPIO\n40mA source\n28mA sink\n1.5A total
 $EndSCHEMATC
